Commit message: FIxes and bug2 added

File: urdf/puzzlebot.urdf (robot description, URDF)
Before this commit: robot Puzzlebot_Jetson_Lidar_Ed., 5 links, 4 joints
Links:
- added link laser_link, mass 0.1; collision cylinder length=0.03 radius=0.035; visual cylinder length=0.03 radius=0.035
- link base_link: mass None -> 2.0; geometry collision box size=0.2 0.2 0.1; visual mesh filename=package://puzzlebot_sim/meshes/Puzzlebot_Jetson_Lidar_Editi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 scale=1 1 1
- link caster_link: mass None -> 0.1; geometry collision sphere radius=0.01; visual mesh filename=package://puzzlebot_sim/meshes/Puzzlebot_Caster_Wheel.stl scale=1 1 1
- link wheel_l_link: mass None -> 0.2; geometry collision cylinder length=0.04 radius=0.05; visual mesh filename=package://puzzlebot_sim/meshes/Puzzlebot_Wheel.stl scale=1 1 1
- link wheel_r_link: mass None -> 0.2; geometry collision cylinder length=0.04 radius=0.05; visual mesh filename=package://puzzlebot_sim/meshes/Puzzlebot_Wheel.stl scale=1 1 1
Joints:
- added joint laser_joint: type fixed, parent base_link, child laser_link, origin xyz=0.0 0.0 0.08 rpy=0 0 0

Commit message: fixes

File: urdf/puzzlebot.urdf (robot description, URDF)
Before this commit: robot puzzlebot, 6 links, 5 joints
Links:
- link base_link: geometry collision box size=0.2 0.2 0.1; visual mesh filename=file:///home/jp/ros2_ws/src/puzzlebot_sim/meshes/Puzzlebot_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 scale=1 1 1
- link caster_link: geometry collision sphere radius=0.01; visual mesh filename=file:///home/jp/ros2_ws/src/puzzlebot_sim/meshes/Puzzlebot_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 scale=1 1 1
- link wheel_l_link: geometry collision cylinder length=0.04 radius=0.05; visual mesh filename=file:///home/jp/ros2_ws/src/puzzlebot_sim/meshes/Puzzlebot_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 scale=1 1 1
- link wheel_r_link: geometry collision cylinder length=0.04 radius=0.05; visual mesh filename=file:///home/jp/ros2_ws/src/puzzlebot_sim/meshes/Puzzlebot_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 scale=1 1 1
